File: wifi-floppy/hardware/wifi_floppy.kicad_sch (KiCad schematic)
At the start: 30 parts, among them J1 Conn_02x17_Odd_Even, J2 Conn_01x04, J3 Conn_01x04, J4 Conn_01x04, Q1 BSS138, Q2 BSS138, Q3 BSS138, Q4 BSS138, Q5 BSS138, Q6 BSS138, Q7 BSS138, Q8 BSS138, U1 RaspberryPi_Pico_W, U2 74LVC541A

Commit message: Add the 22 ohms resistor for the buzzer.
Parts:
- added R12: 22, wifi-floppy-lib:R_1206_3216Metric_Pad1.30x1.75mm_HandSolder, symbol wifi-floppy-lib:R_Small
- BZ1, J1, J2, J3, J4, U1: now not fitted
Connections:
- net +5V: now also R12.1; no longer BZ1.1 (+), Q8.3 (D)
- new net: BZ1.1 (+), Q8.3 (D), R12.2
Changed lines of the file:
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@@
 	)
 	(junction
-		(at 171.45 109.22)
-		(diameter 0)
-		(color 0 0 0 0)
-	)
-	(junction
 		(at 22.86 80.01)
 		(diameter 0)
@@
 	)
 	(junction
+		(at 171.45 109.22)
+		(diameter 0)
+		(color 0 0 0 0)
+	)
+	(junction
 		(at 60.96 31.75)
 		(diameter 0)
@@
 	(wire
 		(pts
+			(xy 171.45 107.95) (xy 171.45 109.22)
+		)
+		(stroke
+			(width 0)
+			(type default)
+		)
+	)
+	(wire
+		(pts
 			(xy 22.86 80.01) (xy 22.86 77.47)
 		)
@@
 		(on_board yes)
 		(in_pos_files yes)
-		(dnp no)
+		(dnp yes)
 		(fields_autoplaced yes)
 		(property "Reference" "J3"
@@
 		(on_board yes)
 		(in_pos_files yes)
-		(dnp no)
+		(dnp yes)
 		(fields_autoplaced yes)
 		(property "Reference" "J2"
@@
 		(on_board yes)
 		(in_pos_files yes)
-		(dnp no)
+		(dnp yes)
 		(fields_autoplaced yes)
 		(property "Reference" "J1"
@@
 		(on_board yes)
 		(in_pos_files yes)
-		(dnp no)
+		(dnp yes)
 		(fields_autoplaced yes)
 		(property "Reference" "J4"
@@
 		(on_board yes)
 		(in_pos_files yes)
-		(dnp no)
+		(dnp yes)
 		(property "Reference" "BZ1"
 			(at 165.1138 114.3578 0)
@@
 		(on_board yes)
 		(in_pos_files yes)
-		(dnp no)
+		(dnp yes)
 		(fields_autoplaced yes)
 		(property "Reference" "U1"
@@
 	)
 	(symbol
+		(lib_id "wifi-floppy-lib:R_Small")
+		(at 171.45 105.41 0)
+		(unit 1)
+		(body_style 1)
+		(exclude_from_sim no)
+		(in_bom yes)
+		(on_board yes)
+		(in_pos_files yes)
+		(dnp no)
+		(fields_autoplaced yes)
+		(property "Reference" "R12"
+			(at 172.9486 104.1978 0)
+			(show_name no)
+			(do_not_autoplace no)
+			(effects
+				(font
+					(size 1.016 1.016)
+				)
+				(justify left)
+			)
+		)
+		(property "Value" "22"
+			(at 172.9486 106.4177 0)
+			(show_name no)
+			(do_not_autoplace no)
+			(effects
+				(font
+					(size 1.27 1.27)
+				)
+				(justify left)
+			)
+		)
+		(property "Footprint" "wifi-floppy-lib:R_1206_3216Metric_Pad1.30x1.75mm_HandSolder"
+			(at 171.45 105.41 0)
+			(hide yes)
+			(show_name no)
+			(do_not_autoplace no)
+			(effects
+				(font
+					(size 1.27 1.27)
+				)
+			)
+		)
+		(property "Datasheet" ""
+			(at 171.45 105.41 0)
+			(hide yes)
+			(show_name no)
+			(do_not_autoplace no)
+			(effects
+				(font
+					(size 1.27 1.27)
+				)
+			)
+		)
+		(property "Description" "Resistor, small symbol"
+			(at 171.45 105.41 0)
+			(hide yes)
+			(show_name no)
+			(do_not_autoplace no)
+			(effects
+				(font
+					(size 1.27 1.27)
+				)
+			)
+		)
+		(property "LCSC" "C2925020"
+			(at 171.45 105.41 0)
+			(hide yes)
+			(show_name no)
+			(do_not_autoplace no)
+			(effects
+				(font
+					(size 1.27 1.27)
+				)
+			)
+		)
+		(pin "1"
+		)
+		(pin "2"
+		)
+		(instances
+			(project "wifi_floppy"
+				(path "/c9178abf-c4d6-4242-b99e-f9f08c77f33c"
+					(reference "R12")
+					(unit 1)
+				)
+			)
+		)
+	)
+	(symbol
 		(lib_id "wifi-floppy-lib:74AHC541")
 		(at 116.84 80.01 0)
@@
 	(symbol
 		(lib_id "power:+5V")
-		(at 171.45 109.22 0)
+		(at 171.45 102.87 0)
 		(unit 1)
 		(body_style 1)
@@
 		(fields_autoplaced yes)
 		(property "Reference" "#PWR028"
-			(at 171.45 113.03 0)
+			(at 171.45 106.68 0)
 			(hide yes)
 			(show_name no)
@@
 		)
 		(property "Value" "+5V"
-			(at 171.45 105.0869 0)
+			(at 171.45 98.7369 0)
 			(show_name no)
 			(do_not_autoplace no)
@@
 		)
 		(property "Footprint" ""
-			(at 171.45 109.22 0)
+			(at 171.45 102.87 0)
 			(hide yes)
 			(show_name no)
@@
 		)
 		(property "Datasheet" ""
-			(at 171.45 109.22 0)
+			(at 171.45 102.87 0)
 			(hide yes)
 			(show_name no)
@@
 		)
 		(property "Description" "Power symbol creates a global label with name \"+5V\""
-			(at 171.45 109.22 0)
+			(at 171.45 102.87 0)
 			(hide yes)
 			(show_name no)

Commit message: Added double footprint for the buzzer (6.5 mm and 5 mm)
Parts:
- BZ1: LCSC DNP -> C2687681
Changed lines of the file:
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@@
 			)
 		)
-		(property "LCSC" "DNP"
+		(property "LCSC" "C2687681"
 			(at 168.91 115.57 0)
 			(hide yes)
